File: kicad/galvoexpress/galvoexpress.kicad_sch (KiCad schematic)
At the start: 12 parts, among them J1 MP1584EN OUT +5V, J2 MP1584EN OUT -, J3 MP1584EN IN +15V, J4 MP1584EN IN -, J5 +15V -15V, J6 laser, J7 Conn_01x09_Pin, J8 0-5V, U1 WEMOS_D1_mini, U2 MCP4922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

Commit message: hele schema
Parts:
- added D1: 1N4006, Diode_THT:D_DO-41_SOD81_P10.16mm_Horizontal, symbol Diode:1N4006
- added J10: laser 2, symbol Connector:Conn_01x03_Pin
- added J9: laser 1, symbol Connector:Conn_01x03_Pin
- added Q1: Q_NPN_BEC, symbol Transistor_BJT:Q_NPN_BEC
- added R1, R3, R4, R6, R7, R9: 10k, symbol Device:R
- added R2: 1k, symbol Device:R
- added R5, R8: 0.5k, symbol Device:R
- added RV1, RV2, RV3, RV4: R_Potentiometer 10k, symbol Device:R_Potentiometer
Connections:
- net at U3.5 (+): now also RV2.1
- net at U3.6 (-): now also R4.2, RV1.2
- net at U3.7: now also J9.3 (Pin_3), R1.1, RV1.3
- net at J8.1 (Pin_1), U1.9 (5V): now also J6.1 (Pin_1), D1.1 (K); no longer J1.1 (Pin_1), J1.2 (Pin_2)
- net at J2.1 (Pin_1), J2.2 (Pin_2), J4.1 (Pin_1)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: now also J10.1 (Pin_1), J9.1 (Pin_1), Q1.3 (C), R4.1, R5.1, R6.1, R8.1
- net at U1.12 (D3): now also R2.1
- net at U4.4 (V-): now also J5.3 (Pin_3), U3.4 (V-)
- net at U4.5 (+): now also R8.2
- net at U4.6 (-): now also R7.2, R9.1
- net at U4.7: now also J10.2 (Pin_2), R9.2
- net at U4.1: now also J10.3 (Pin_3), R7.1, RV4.3
- net at U4.2 (-): now also R6.2, RV4.2
- net at U4.3 (+): now also RV3.1
- net at U2.13 (VrefA): now also RV2.2
- net at U2.14 (VA): now also RV3.2
- net at U3.1: now also J9.2 (Pin_2), R3.2
- net at U3.2 (-): now also R1.2, R3.1
- net at U3.3 (+): now also R5.2
- net at J6.3 (Pin_3): now also Q1.2 (E)
- new net: D1.2 (A), J1.1 (Pin_1), J1.2 (Pin_2)
- new net: Q1.1 (B), R2.2
Other:
- moved on the sheet: J6, U3A, U3B, U3C, U4A, U4B, U4C

Commit message: kicad WIP
Parts:
- removed J7: Conn_01x09_Pin, symbol Connector:Conn_01x09_Pin
- removed J8: 0-5V, symbol Connector:Conn_01x02_Pin
- removed RV1, RV2, RV3, RV4: R_Potentiometer 10k, symbol Device:R_Potentiometer
- added J7: Screw_Terminal_01x02 5V, TerminalBlock_MetzConnect:TerminalBlock_MetzConnect_Type059_RT06302HBWC_1x02_P3.50mm_Horizontal, symbol Connector:Screw_Terminal_01x02
- added J8: Screw_Terminal_01x08, TerminalBlock_Phoenix:TerminalBlock_Phoenix_MPT-0,5-8-2.54_1x08_P2.54mm_Horizontal, symbol Connector:Screw_Terminal_01x08
- added RV1, RV2, RV3, RV6: R_Potentiometer_Trim 10k, Potentiometer_THT:Potentiometer_Bourns_3296W_Vertical, symbol Device:R_Potentiometer_Trim
- J1, J2, J3, J4: footprint (none) -> Connector_PinHeader_2.54mm:PinHeader_1x02_P2.54mm_Vertical
- J10, J5, J9: footprint (none) -> Connector_JST:JST_XH_S3B-XH-A-1_1x03_P2.50mm_Horizontal
- J6: footprint (none) -> Connector_PinHeader_2.54mm:PinHeader_1x03_P2.54mm_Vertical
- Q1: footprint (none) -> Package_TO_SOT_THT:TO-92L_Inline
- R1, R2, R3, R4, R5, R6, R7, R8, R9: footprint (none) -> Resistor_THT:R_Axial_DIN0309_L9.0mm_D3.2mm_P12.70mm_Horizontal
- U2: footprint (none) -> Package_DIP:DIP-14_W7.62mm
- U3, U4: footprint (none) -> Package_DIP:DIP-8_W7.62mm
Connections:
- net at U3.5 (+): now also RV6.1
- net at R4.2, U3.6 (-): now also RV1.2
- net at J9.3 (Pin_3), R1.1, U3.7: now also RV1.3
- net at J10.1 (Pin_1), J2.1 (Pin_1), J2.2 (Pin_2)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: now also J7.1 (Pin_1)
- net at D1.1 (K), J6.1 (Pin_1), U1.9 (5V): now also J7.2 (Pin_2)
- net at J10.3 (Pin_3), R7.1, U4.1: now also RV3.3
- net at U4.3 (+): now also RV2.1
- net at U2.14 (VA): now also RV2.2
- net at U1.11 (D4): now also J8.7 (Pin_7)
- net at U1.13 (SDA/D2): now also J8.6 (Pin_6)
- net at U1.14 (SCL/D1): now also J8.5 (Pin_5)
- net at U1.15 (RX): now also J8.2 (Pin_2)
- net at U1.16 (TX): now also J8.1 (Pin_1)
- net at U1.2 (A0): now also J8.3 (Pin_3)
- net at U1.3 (D0): now also J8.4 (Pin_4)
- net at U1.5 (MISO/D6): now also J8.8 (Pin_8)
- net at R1.2, U3.2 (-): now also R3.2; no longer R3.1
- net at J9.2 (Pin_2), U3.1: now also R3.1; no longer R3.2
- net at R6.2, U4.2 (-): now also RV3.2
- net at U2.13 (VrefA): now also RV6.2

Commit message: kicad v1.0
Connections:
- net at R1.1, RV1.3, U3.7: now also J9.1 (Pin_1); no longer J9.3 (Pin_3)
- net at J2.1 (Pin_1), J2.2 (Pin_2), J4.1 (Pin_1)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: now also J10.3 (Pin_3), J9.3 (Pin_3); no longer J10.1 (Pin_1), J9.1 (Pin_1)
- net at R7.1, RV3.3, U4.1: now also J10.1 (Pin_1); no longer J10.3 (Pin_3)
- net at U1.11 (D4): now also J8.8 (Pin_8); no longer J8.7 (Pin_7)
- net at U1.13 (SDA/D2): now also J8.7 (Pin_7); no longer J8.6 (Pin_6)
- net at U1.14 (SCL/D1): now also J8.6 (Pin_6); no longer J8.5 (Pin_5)
- net at U1.15 (RX): now also J8.5 (Pin_5); no longer J8.2 (Pin_2)
- net at U1.16 (TX): now also J8.4 (Pin_4); no longer J8.1 (Pin_1)
- net at U1.2 (A0): now also J8.1 (Pin_1); no longer J8.3 (Pin_3)
- net at U1.3 (D0): now also J8.2 (Pin_2); no longer J8.4 (Pin_4)
- net at U1.5 (MISO/D6): now also J8.3 (Pin_3); no longer J8.8 (Pin_8)

Commit message: kicad repairs
Connections:
- net at J10.3 (Pin_3), J2.1 (Pin_1), J2.2 (Pin_2)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: now also Q1.1 (B), U2.8 (~{LDAC}); no longer Q1.3 (C)
- net at RV2.2: now also U2.10 (VB); no longer U2.14 (VA)
- net at RV6.2: now also U2.14 (VA); no longer U2.13 (VrefA)
- net at U1.7 (CS/D8), U2.3 (~{CS}): no longer U2.8 (~{LDAC})
- net at U1.8 (3V3), U2.1 (Vdd), U2.9 (~{SHDN}): now also U2.11 (VrefB), U2.13 (VrefA)
- net at R2.2: now also Q1.2 (E); no longer Q1.1 (B)
- net at J6.3 (Pin_3): now also Q1.3 (C); no longer Q1.2 (E)
Other:
- moved on the sheet: R2
